Commit message: Added robot urdf data

File: data/2dof_planar_arm.urdf (robot description, URDF)
Before this commit: robot 2dof_arm, 3 links, 2 joints
Links:
- link base: geometry visual cylinder length=0.1 radius=0.05
- link link1: geometry visual box size=0.5 0.05 0.05
- link link2: geometry visual box size=0.4 0.05 0.05
Joints:
- joint joint1: axis (none) -> 0 0 1; origin (none) -> xyz=0 0 0.1 rpy=0 0 0
- joint joint2: axis (none) -> 0 0 1; limit (none) -> lower=-3.14 upper=3.14; origin (none) -> xyz=0.5 0 0 rpy=0 0 0
